File: schematic/SensorNode/V1_0/sensorNodev1_0.brd (EAGLE design)
At the start: 62.9 x 84.7 mm, 34 parts, among them IC1 V_REG_MIC2920, IC2 SI7021-A10-GM, J1 AVR_SPI_PRG_62X3_LOCK, U1 ATMEGA328P_TQFP, U2 ADA4077-1ARZ

Commit message: Replacing Screen connector with low profile Jst-EH connector
Parts:
- SCREEN: value (none) -> JST-B5B-EH-A; device SparkFun-Connectors:1X05 -> bespin:JST-B5B-ED-A
- moved SCREEN 2.73 mm to (0.40, 46.6), turned to 0 degrees
- renumbered IC2 to OPAMP_CO, JP3 to CO2
Connections:
- net GND: now also SCREEN.5; no longer SCREEN.1
- net SDA: now also SCREEN.2; no longer SCREEN.4
- net VCC: now also SCREEN.1; no longer SCREEN.5
Routing:
- net GND: track 20.9 -> 39.1 mm, vias 0 -> 1
- net SDA: track 43.4 -> 44.3 mm
Changed lines of the file:
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@@
 <attribute name="VALUE" x="4.206" y="29.3395" size="0.4064" layer="27" rot="R180"/>
 </element>
-<element name="JP3" library="bespin" package="K-30" value="K-30K-30" x="59" y="10.959" smashed="yes" rot="R90">
+<element name="CO2" library="bespin" package="K-30" value="K-30K-30" x="59" y="10.959" smashed="yes" rot="R90">
 <attribute name="NAME" x="52.0912" y="11.5178" size="1.27" layer="25" ratio="10" rot="R90"/>
 <attribute name="VALUE" x="52.015" y="21.119" size="1.27" layer="27" rot="R90"/>
-</element>
-<element name="SCREEN" library="SparkFun-Connectors" package="1X05" value="" x="2.346" y="48.517" smashed="yes" rot="R90">
-<attribute name="NAME" x="6.2322" y="47.6788" size="1.27" layer="25" ratio="10" rot="R90"/>
-<attribute name="VALUE" x="5.521" y="47.247" size="1.27" layer="27" rot="R90"/>
 </element>
 <element name="ENTER" library="SparkFun-Electromechanical" package="TACTILE-PTH" value="SWITCH-MOMENTARY-2PTH" x="46.99" y="5.08"/>
@@
 <element name="U$3" library="bespin" package="DUPPY_LOGO" value="" x="49" y="55" rot="MR270"/>
 <element name="U$4" library="bespin" package="CONTAINER_BOTTOM" value="" x="-3" y="-2"/>
-<element name="IC2" library="bespin" package="DFN6-3X3" value="SI7021-A10-GM" x="5" y="64">
+<element name="OPAMP_CO" library="bespin" package="DFN6-3X3" value="SI7021-A10-GM" x="5" y="64">
 <attribute name="OC_NEWARK" value="55X3111" x="5" y="64" size="1.778" layer="27" display="off"/>
 <attribute name="MPN" value="Si7021-A10-GM" x="5" y="64" size="1.778" layer="27" display="off"/>
@@
 <attribute name="OC_FARNELL" value="2422571" x="5" y="64" size="1.778" layer="27" display="off"/>
 </element>
+<element name="SCREEN" library="bespin" package="JST-B5B-ED-A" value="JST-B5B-EH-A" x="0.4" y="46.6"/>
 </elements>
 <signals>
@@
 <vertex x="-1" y="0"/>
 </polygon>
-<contactref element="SCREEN" pad="5"/>
 <contactref element="R2" pad="2"/>
 <contactref element="R6" pad="2"/>
@@
 <wire x1="25.3622" y1="64.635" x2="37.29" y2="64.635" width="0.254" layer="1"/>
 <wire x1="37.29" y1="64.635" x2="37.89" y2="64.035" width="0.254" layer="1"/>
-<contactref element="IC2" pad="5"/>
-<wire x1="2.346" y1="58.677" x2="4.677" y2="58.677" width="0.254" layer="1"/>
-<wire x1="4.677" y1="58.677" x2="8" y2="62" width="0.254" layer="1"/>
-<wire x1="8" y1="62" x2="8" y2="64" width="0.254" layer="1"/>
-<wire x1="8" y1="64" x2="6.45" y2="64" width="0.254" layer="1"/>
+<contactref element="OPAMP_CO" pad="5"/>
+<contactref element="SCREEN" pad="1"/>
+<wire x1="2.305" y1="58.5888" x2="5.5888" y2="58.5888" width="0.254" layer="1"/>
+<wire x1="5.5888" y1="58.5888" x2="8" y2="61" width="0.254" layer="1"/>
+<wire x1="8" y1="61" x2="8" y2="63" width="0.254" layer="1"/>
+<wire x1="8" y1="63" x2="7" y2="64" width="0.254" layer="1"/>
+<wire x1="7" y1="64" x2="6.45" y2="64" width="0.254" layer="1"/>
 </signal>
 <signal name="GND">
@@
 <vertex x="61.88" y="84.74"/>
 </polygon>
-<contactref element="JP3" pad="14"/>
-<contactref element="SCREEN" pad="1"/>
+<contactref element="CO2" pad="14"/>
 <contactref element="ENTER" pad="3"/>
 <contactref element="BACK" pad="3"/>
@@
 <wire x1="6.3" y1="44.6" x2="2.514" y2="44.6" width="0.254" layer="16"/>
 <wire x1="2.514" y1="44.6" x2="2.381" y2="44.733" width="0.254" layer="16"/>
-<wire x1="2.381" y1="44.733" x2="2.381" y2="48.482" width="0.254" layer="16"/>
-<wire x1="2.381" y1="48.482" x2="2.346" y2="48.517" width="0.254" layer="16"/>
 <contactref element="J1" pad="6"/>
 <contactref element="U$1" pad="CE"/>
@@
 <contactref element="U$1" pad="CE1"/>
 <contactref element="U2" pad="3"/>
-<contactref element="IC2" pad="2"/>
+<contactref element="OPAMP_CO" pad="2"/>
+<contactref element="SCREEN" pad="5"/>
+<wire x1="2.381" y1="44.733" x2="2.305" y2="44.733" width="0.254" layer="16"/>
+<wire x1="2.305" y1="44.733" x2="2.305" y2="48.6066" width="0.254" layer="16"/>
+<wire x1="3.55" y1="64" x2="3" y2="64" width="0.254" layer="1"/>
+<wire x1="3" y1="64" x2="2" y2="63" width="0.254" layer="1"/>
+<wire x1="2" y1="63" x2="2" y2="62" width="0.254" layer="1"/>
+<via x="2" y="62" extent="1-16" drill="0.6"/>
+<wire x1="2" y1="62" x2="0" y2="60" width="0.254" layer="16"/>
+<wire x1="0" y1="60" x2="0" y2="50.9116" width="0.254" layer="16"/>
+<wire x1="0" y1="50.9116" x2="2.305" y2="48.6066" width="0.254" layer="16"/>
 </signal>
 <signal name="RX">
@@
 </signal>
 <signal name="SDA">
-<contactref element="SCREEN" pad="4"/>
 <contactref element="U1" pad="27"/>
 <wire x1="29.4474" y1="43.49" x2="26.01" y2="43.49" width="0.254" layer="1"/>
 <wire x1="26.01" y1="43.49" x2="13.5" y2="56" width="0.254" layer="1"/>
-<wire x1="13.5" y1="56" x2="2.483" y2="56" width="0.254" layer="1"/>
-<wire x1="2.483" y1="56" x2="2.346" y2="56.137" width="0.254" layer="1"/>
-<contactref element="IC2" pad="1"/>
-<wire x1="2.346" y1="56.137" x2="2.263" y2="56.137" width="0.254" layer="1"/>
-<wire x1="2.263" y1="56.137" x2="0.8" y2="57.1" width="0.254" layer="1"/>
-<wire x1="0.8" y1="57.1" x2="0.8" y2="62.75" width="0.254" layer="1"/>
-<wire x1="0.8" y1="62.75" x2="3.55" y2="65" width="0.254" layer="1"/>
+<contactref element="OPAMP_CO" pad="1"/>
+<wire x1="0.8" y1="56.0996" x2="0.8" y2="62.8" width="0.254" layer="1"/>
+<contactref element="SCREEN" pad="2"/>
+<wire x1="13.5" y1="56" x2="2.305" y2="56" width="0.254" layer="1"/>
+<wire x1="2.305" y1="56" x2="2.305" y2="56.0996" width="0.254" layer="1"/>
+<wire x1="2.305" y1="56.0996" x2="0.8" y2="56.0996" width="0.254" layer="1"/>
+<wire x1="0.8" y1="62.8" x2="3" y2="65" width="0.254" layer="1"/>
+<wire x1="3" y1="65" x2="3.55" y2="65" width="0.254" layer="1"/>
 </signal>
 <signal name="SCL">
-<contactref element="SCREEN" pad="3"/>
 <contactref element="U1" pad="28"/>
 <wire x1="29.4474" y1="42.69" x2="25.31" y2="42.69" width="0.254" layer="1"/>
 <wire x1="25.31" y1="42.69" x2="14.4" y2="53.6" width="0.254" layer="1"/>
-<wire x1="14.4" y1="53.6" x2="2.349" y2="53.6" width="0.254" layer="1"/>
-<wire x1="2.349" y1="53.6" x2="2.346" y2="53.597" width="0.254" layer="1"/>
-<contactref element="IC2" pad="6"/>
-<wire x1="2.349" y1="53.6" x2="0.1" y2="53.6" width="0.254" layer="1"/>
-<wire x1="0.1" y1="53.6" x2="0.1" y2="63.6" width="0.254" layer="1"/>
+<contactref element="OPAMP_CO" pad="6"/>
 <wire x1="0.1" y1="63.6" x2="3" y2="66" width="0.254" layer="1"/>
 <wire x1="3" y1="66" x2="6.45" y2="66" width="0.254" layer="1"/>
 <wire x1="6.45" y1="66" x2="6.45" y2="65" width="0.254" layer="1"/>
+<contactref element="SCREEN" pad="3"/>
+<wire x1="14.4" y1="53.6" x2="2.305" y2="53.6" width="0.254" layer="1"/>
+<wire x1="2.305" y1="53.6" x2="2.305" y2="53.6104" width="0.254" layer="1"/>
+<wire x1="2.305" y1="53.6104" x2="0.1" y2="53.6104" width="0.254" layer="1"/>
+<wire x1="0.1" y1="53.6104" x2="0.1" y2="63.6" width="0.254" layer="1"/>
 </signal>
 <signal name="5V">
@@
 <contactref element="IC1" pad="1"/>
 <contactref element="C1" pad="1"/>
-<contactref element="JP3" pad="17"/>
+<contactref element="CO2" pad="17"/>
 <wire x1="21.13" y1="32.62" x2="24.38" y2="32.62" width="0.254" layer="16"/>
 <wire x1="24.38" y1="32.62" x2="26" y2="31" width="0.254" layer="16"/>
@@
 </signal>
 <signal name="TX_K30">
-<contactref element="JP3" pad="27"/>
+<contactref element="CO2" pad="27"/>
 <contactref element="U1" pad="2"/>
 <wire x1="31.74" y1="37.9974" x2="31.74" y2="36.26" width="0.254" layer="1"/>
@@
 </signal>
 <signal name="RX_K30">
-<contactref element="JP3" pad="26"/>
+<contactref element="CO2" pad="26"/>
 <contactref element="U1" pad="1"/>
 <wire x1="30.94" y1="37.9974" x2="30.94" y2="37.94" width="0.254" layer="1"/>
